Commit message: scaled wheel mesh and added base_link stl file

File: duda_robot/src/duda_description/urdf/wheel.urdf.xacro (robot description, xacro)
@@ -11,5 +11,5 @@
 				<origin xyz="0 0 0" rpy="0 0 0" />
 				<geometry>
-					<mesh filename="package://duda_description/meshes/wheel.dae" />
+					<mesh filename="package://duda_description/meshes/wheel.dae" scale="5 5 5"/>
 				</geometry>
 			</visual>
