Commit message: changes for first implementation

File: duda_robot/src/duda_description/urdf/duda.urdf.xacro (robot description, xacro)
@@ -1,8 +1,8 @@
 <?xml version="1.0"?>
 <robot name="duda" xmlns:xacro="http://ros.org/wiki/xacro">
-    <link name = "base_model">
+    <link name = "base_link">
         <visual>
             <geometry>
-                <box size="0.6 0.1 0.2"/>
+                <box size="2.6 0.1 0.2"/>
             </geometry>
         </visual>

Commit message: xacro:macro implementation

File: duda_robot/src/duda_description/urdf/duda.urdf.xacro (robot description, xacro)
@@ -1,10 +1,13 @@
 <?xml version="1.0"?>
 <robot name="duda" xmlns:xacro="http://ros.org/wiki/xacro">
-    <link name = "base_link">
-        <visual>
-            <geometry>
-                <box size="2.6 0.1 0.2"/>
-            </geometry>
-        </visual>
-    </link>
+    <xacro:macro name="compartment" params="name length width height">
+        <link name="${name}">
+            <visual>
+                <geometry>
+                    <box size = "${length} ${width} ${height}">
+                </geometry>
+            </visual>
+        </link>
+    </xacro:macro>
+    <xacro:compartment name="base_link" length="2.6" width="0.4" height="0.4" />
 </robot>

Commit message: link with xacro property

File: duda_robot/src/duda_description/urdf/duda.urdf.xacro (robot description, xacro)
@@ -1,13 +1,30 @@
 <?xml version="1.0"?>
 <robot name="duda" xmlns:xacro="http://ros.org/wiki/xacro">
-    <xacro:macro name="compartment" params="name length width height">
-        <link name="${name}">
-            <visual>
-                <geometry>
-                    <box size = "${length} ${width} ${height}">
-                </geometry>
-            </visual>
-        </link>
-    </xacro:macro>
-    <xacro:compartment name="base_link" length="2.6" width="0.4" height="0.4" />
+     <!-- Include Materials -->
+     <material name="Black">
+         <color rgba="0.0 0.0 0.0 1.0"/>
+     </material>
+     <material name="Red">
+         <color rgba="0.8 0.0 0.0 1.0"/>
+     </material>
+     <material name="White">
+         <color rgba="1 1 1 1"/>
+     </material>
+     <!-- Middle Compartment Dimensions -->
+     <xacro:property name="middle_comp_length" value="2.6" />
+     <xacro:property name="middle_comp_width" value="0.6" />
+     <xacro:property name="middle_comp_length" value="0.4" />
+     <!-- Front Compartment Dimensions -->
+     <xacro:property name="front_comp_length" value="1.6" />
+     <xacro:property name="front_comp_width" value="0.6" />
+     <xacro:property name="front_comp_length" value="0.4" />
+    <link name="base_link">
+        <visual>
+            <origin xyz="0.0 0.0 0.0" rpy="0.0 0.0 0.0"/>
+            <geometry>
+                <box size="${middle_comp_length} ${middle_comp_width} ${middle_comp_height}"/>
+            </geometry>
+            <material name="Black" />
+        </visual>
+    </link>
 </robot>

Commit message: added front compartment and joint

File: duda_robot/src/duda_description/urdf/duda.urdf.xacro (robot description, xacro)
@@ -14,9 +14,10 @@
      <xacro:property name="middle_comp_length" value="2.6" />
      <xacro:property name="middle_comp_width" value="0.6" />
-     <xacro:property name="middle_comp_length" value="0.4" />
+     <xacro:property name="middle_comp_height" value="0.4" />
      <!-- Front Compartment Dimensions -->
      <xacro:property name="front_comp_length" value="1.6" />
      <xacro:property name="front_comp_width" value="0.6" />
-     <xacro:property name="front_comp_length" value="0.4" />
+     <xacro:property name="front_comp_height" value="0.4" />
+    <!-- Base link / Middle Compartment -->
     <link name="base_link">
         <visual>
@@ -28,3 +29,18 @@
         </visual>
     </link>
+    <!-- Front link / Front Compartment -->
+    <link name="front_link">
+        <visual>
+            <origin xyz="0.0 0.0 0.0" rpy="0.0 0.0 0.0"/>
+            <geometry>
+                <box size="${front_comp_length} ${front_comp_width} ${front_comp_height}"/>
+            </geometry>
+            <material name="Black" />
+        </visual>
+    </link>
+    <joint name="base_front_joint" type="fixed">
+        <origin xyz="2.6 0 0" rpy="0 0 0" />
+        <parent link="base_link"/>
+        <child link="front_link"/>
+    </joint>
 </robot>

Commit message: changes made in imp pc

File: duda_robot/src/duda_description/urdf/duda.urdf.xacro (robot description, xacro)
@@ -17,5 +17,5 @@
      <!-- Front Compartment Dimensions -->
      <xacro:property name="front_comp_length" value="1.6" />
-     <xacro:property name="front_comp_width" value="0.6" />
+     <xacro:property name="front_comp_width" value="5.6" />
      <xacro:property name="front_comp_height" value="0.4" />
     <!-- Base link / Middle Compartment -->

Commit message: automatic xacro to urdf conversion in launch and xacro fine tuning for rviz

File: duda_robot/src/duda_description/urdf/duda.urdf.xacro (robot description, xacro)
@@ -32,5 +32,5 @@
     <link name="front_link">
         <visual>
-            <origin xyz="0.0 0.0 0.0" rpy="0.0 0.0 0.0"/>
+            <origin xyz="0.8 0.0 0.0" rpy="0.0 0.0 0.0"/>
             <geometry>
                 <box size="${front_comp_length} ${front_comp_width} ${front_comp_height}"/>
@@ -40,5 +40,5 @@
     </link>
     <joint name="base_front_joint" type="fixed">
-        <origin xyz="2.6 0 0" rpy="0 0 0" />
+        <origin xyz="1.3 0 0" rpy="0 0 0" />
         <parent link="base_link"/>
         <child link="front_link"/>

Commit message: added wheel to duda

File: duda_robot/src/duda_description/urdf/duda.urdf.xacro (robot description, xacro)
@@ -11,4 +11,8 @@
          <color rgba="1 1 1 1"/>
      </material>
+     <!--Include URDF/XACRO files -->
+     <xacro:include filename="$(find duda_description)/urdf/wheel.urdf.xacro" />
+     <!-- Constants -->
+     <xacro:property name="M_PI" value="3.14159"/>
      <!-- Middle Compartment Dimensions -->
      <xacro:property name="middle_comp_length" value="2.6" />
@@ -19,4 +23,7 @@
      <xacro:property name="front_comp_width" value="5.6" />
      <xacro:property name="front_comp_height" value="0.4" />
+    <!-- Wheel Properties -->
+    <xacro:property name="wheel_length" value="0.1143" />
+    <xacro:property name="wheel_radius" value="0.1651" />
     <!-- Base link / Middle Compartment -->
     <link name="base_link">
@@ -44,3 +51,7 @@
         <child link="front_link"/>
     </joint>
+     <!-- duda wheel macros -->
+    <xacro:duda_wheel wheel_prefix="front_left">
+        <origin xyz="0 0 0" rpy="0 0 0" />
+    </xacro:duda_wheel>
 </robot>

Commit message: added base_link mesh to visual and the wheels

File: duda_robot/src/duda_description/urdf/duda.urdf.xacro (robot description, xacro)
@@ -23,5 +23,9 @@
      <xacro:property name="front_comp_width" value="5.6" />
      <xacro:property name="front_comp_height" value="0.4" />
-    <!-- Wheel Properties -->
+    <!-- Wheel Mounting Positions -->
+    <xacro:property name="wheelbase" value="0.5120" />
+    <xacro:property name="track" value="64.5" />
+    <xacro:property name="wheel_vertical_offset" value="0.03282" />
+    <!-- Wheel Properties for Collision -->
     <xacro:property name="wheel_length" value="0.1143" />
     <xacro:property name="wheel_radius" value="0.1651" />
@@ -31,27 +35,15 @@
             <origin xyz="0.0 0.0 0.0" rpy="0.0 0.0 0.0"/>
             <geometry>
-                <box size="${middle_comp_length} ${middle_comp_width} ${middle_comp_height}"/>
+                <mesh filename="package://duda_description/meshes/base_link.stl" scale="1 1 1"/>
             </geometry>
             <material name="Black" />
         </visual>
     </link>
-    <!-- Front link / Front Compartment -->
-    <link name="front_link">
-        <visual>
-            <origin xyz="0.8 0.0 0.0" rpy="0.0 0.0 0.0"/>
-            <geometry>
-                <box size="${front_comp_length} ${front_comp_width} ${front_comp_height}"/>
-            </geometry>
-            <material name="Black" />
-        </visual>
-    </link>
-    <joint name="base_front_joint" type="fixed">
-        <origin xyz="1.3 0 0" rpy="0 0 0" />
-        <parent link="base_link"/>
-        <child link="front_link"/>
-    </joint>
-     <!-- duda wheel macros -->
+     <!-- Duda wheel macros -->
     <xacro:duda_wheel wheel_prefix="front_left">
-        <origin xyz="0 0 0" rpy="0 0 0" />
+        <origin xyz="0 ${track/2} 0" rpy="0 0 0" />
+    </xacro:duda_wheel>
+    <xacro:duda_wheel wheel_prefix="front_right">
+        <origin xyz="0 ${-track/2} 0" rpy="0 0 0" />
     </xacro:duda_wheel>
 </robot>

File: duda_robot/src/duda_description/urdf/wheel.urdf.xacro (robot description, xacro)
@@ -11,5 +11,5 @@
 				<origin xyz="0 0 0" rpy="0 0 0" />
 				<geometry>
-					<mesh filename="package://duda_description/meshes/wheel.dae" scale="5 5 5"/>
+					<mesh filename="package://duda_description/meshes/wheel.dae" scale="2.5 2.5 2.5"/>
 				</geometry>
 			</visual>

Commit message: track value updated

File: duda_robot/src/duda_description/urdf/duda.urdf.xacro (robot description, xacro)
@@ -25,5 +25,5 @@
     <!-- Wheel Mounting Positions -->
     <xacro:property name="wheelbase" value="0.5120" />
-    <xacro:property name="track" value="64.5" />
+    <xacro:property name="track" value="0.645" />
     <xacro:property name="wheel_vertical_offset" value="0.03282" />
     <!-- Wheel Properties for Collision -->

Commit message: middle compartment

File: duda_robot/src/duda_description/urdf/duda.urdf.xacro (robot description, xacro)
@@ -35,5 +35,5 @@
             <origin xyz="0.0 0.0 0.0" rpy="0.0 0.0 0.0"/>
             <geometry>
-                <mesh filename="package://duda_description/meshes/base_link.stl" scale="1 1 1"/>
+                <box size="0.480 0.631 0.355"/>
             </geometry>
             <material name="Black" />

Commit message: after network sharing

File: duda_robot/src/duda_description/urdf/duda.urdf.xacro (robot description, xacro)
@@ -3,8 +3,14 @@
      <!-- Include Materials -->
      <material name="Black">
-         <color rgba="0.0 0.0 0.0 1.0"/>
+         <color rgba="0.0 0.0 0.0 0.6"/>
      </material>
      <material name="Red">
-         <color rgba="0.8 0.0 0.0 1.0"/>
+         <color rgba="0.8 0.0 0.0 0.6"/>
+     </material>
+    <material name="Yellow">
+         <color rgba="0.8 0.8 0.0 0.6"/>
+     </material>
+     <material name="Blue">
+         <color rgba="0.0 0.0 0.4 0.6"/>
      </material>
      <material name="White">
@@ -16,11 +22,17 @@
      <xacro:property name="M_PI" value="3.14159"/>
      <!-- Middle Compartment Dimensions -->
-     <xacro:property name="middle_comp_length" value="2.6" />
-     <xacro:property name="middle_comp_width" value="0.6" />
-     <xacro:property name="middle_comp_height" value="0.4" />
+     <xacro:property name="middle_comp_length" value="0.480" />
+     <xacro:property name="middle_comp_width" value="0.630" />
+     <xacro:property name="middle_comp_height" value="0.355" />
      <!-- Front Compartment Dimensions -->
-     <xacro:property name="front_comp_length" value="1.6" />
-     <xacro:property name="front_comp_width" value="5.6" />
-     <xacro:property name="front_comp_height" value="0.4" />
+     <xacro:property name="front_comp_length" value="0.415" />
+     <xacro:property name="front_comp_width" value="0.520" />
+     <xacro:property name="front_comp_height" value="0.265" />
+     <!-- Rear Compartment Dimensions -->
+     <xacro:property name="rear_comp_length" value="0.325" />
+     <xacro:property name="rear_comp_width" value="0.520" />
+     <xacro:property name="rear_comp_height" value="0.265" />
+    <!-- LiDAR Dimensions -->
+     <xacro:property name="lidar_depth" value="0.098" />
     <!-- Wheel Mounting Positions -->
     <xacro:property name="wheelbase" value="0.5120" />
@@ -30,20 +42,76 @@
     <xacro:property name="wheel_length" value="0.1143" />
     <xacro:property name="wheel_radius" value="0.1651" />
+    <!-- Map -->
+    <link name="map">
+    </link>
     <!-- Base link / Middle Compartment -->
     <link name="base_link">
         <visual>
-            <origin xyz="0.0 0.0 0.0" rpy="0.0 0.0 0.0"/>
             <geometry>
-                <box size="0.480 0.631 0.355"/>
+                <box size="${middle_comp_length} ${middle_comp_width} ${middle_comp_height}"/>
             </geometry>
             <material name="Black" />
         </visual>
     </link>
+    <!-- Map to base joint -->
+    <joint name="map_to_base" type="fixed">
+        <parent link="map"/>
+        <child link="base_link"/>
+        <origin xyz="0 0 ${middle_comp_height/2}"/>
+    </joint>
+    <!-- Front link / Front Compartment -->
+    <link name="front_link">
+        <visual>
+            <origin xyz="${front_comp_length/2} 0.0 0.0" rpy="0.0 0.0 0.0"/>
+            <geometry>
+                <box size="${front_comp_length} ${front_comp_width} ${front_comp_height}"/>
+            </geometry>
+            <material name="Blue" />
+        </visual>
+    </link>
+    <!-- Base-Front Join -->
+    <joint name="base_to_front" type="fixed">
+        <parent link="base_link"/>
+        <child link="front_link"/>
+        <origin xyz="${middle_comp_length/2} 0.0 0.0"/>
+    </joint>
+    <!-- Rear link / Rear Compartment -->
+    <link name="rear_link">
+        <visual>
+            <origin xyz="${-(rear_comp_length/2)} 0.0 0.0" rpy="0.0 0.0 0.0"/>
+            <geometry>
+                <box size="${rear_comp_length} ${rear_comp_width} ${rear_comp_height}"/>
+            </geometry>
+            <material name="Yellow" />
+        </visual>
+    </link>
+    <!-- Base-Rear Join -->
+    <joint name="base_to_rear" type="fixed">
+        <parent link="base_link"/>
+        <child link="rear_link"/>
+        <origin xyz="${-(middle_comp_length/2)} 0.0 0.0"/>
+    </joint>
+    <!-- LiDAR Link -->
+    <link name="lidar_link">
+        <visual>
+            <origin xyz="${lidar_depth/2} 0.0 0.0" rpy="0.0 0.0 ${-radians(90)}"/>
+            <geometry>
+                <mesh filename="package://duda_description/meshes/lidar.stl" scale="0.001 0.001 0.001"/>
+            </geometry>
+            <material name="Red" />
+        </visual>
+    </link>
+    <!-- front-lidar Joint -->
+    <joint name="front_to_lidar" type="fixed">
+        <parent link="front_link"/>
+        <child link="lidar_link"/>
+        <origin xyz="${front_comp_length} 0.0 0.0"/>
+    </joint>
      <!-- Duda wheel macros -->
     <xacro:duda_wheel wheel_prefix="front_left">
-        <origin xyz="0 ${track/2} 0" rpy="0 0 0" />
+        <origin xyz="${front_comp_length/2} ${track/2} ${-(front_comp_height/2)}" rpy="0 0 0" />
     </xacro:duda_wheel>
     <xacro:duda_wheel wheel_prefix="front_right">
-        <origin xyz="0 ${-track/2} 0" rpy="0 0 0" />
+        <origin xyz="${front_comp_length/2} ${-track/2} ${-(front_comp_height/2)}" rpy="0 0 0" />
     </xacro:duda_wheel>
 </robot>

File: duda_robot/src/duda_description/urdf/wheel.urdf.xacro (robot description, xacro)
@@ -11,5 +11,5 @@
 				<origin xyz="0 0 0" rpy="0 0 0" />
 				<geometry>
-					<mesh filename="package://duda_description/meshes/wheel.dae" scale="2.5 2.5 2.5"/>
+					<mesh filename="package://duda_description/meshes/wheel.dae" scale="0.75 0.75 0.75"/>
 				</geometry>
 			</visual>
@@ -29,5 +29,5 @@
 		</gazebo>
 		<joint name="${wheel_prefix}_wheel" type="continuous">
-			<parent link="base_link"/>
+			<parent link="front_link"/>
 			<child link="${wheel_prefix}_wheel_link"/>
 			<xacro:insert_block name="joint_pose"/>

Commit message: urdf with base mesh

File: duda_robot/src/duda_description/urdf/duda.urdf.xacro (robot description, xacro)
@@ -21,33 +21,39 @@
      <!-- Constants -->
      <xacro:property name="M_PI" value="3.14159"/>
-     <!-- Middle Compartment Dimensions -->
-     <xacro:property name="middle_comp_length" value="0.480" />
-     <xacro:property name="middle_comp_width" value="0.630" />
-     <xacro:property name="middle_comp_height" value="0.355" />
-     <!-- Front Compartment Dimensions -->
-     <xacro:property name="front_comp_length" value="0.415" />
-     <xacro:property name="front_comp_width" value="0.520" />
-     <xacro:property name="front_comp_height" value="0.265" />
-     <!-- Rear Compartment Dimensions -->
-     <xacro:property name="rear_comp_length" value="0.325" />
-     <xacro:property name="rear_comp_width" value="0.520" />
-     <xacro:property name="rear_comp_height" value="0.265" />
+     <!-- Base_Link Visual Offsets -->
+     <xacro:property name="base_long_offset" value="-0.61" />
+     <xacro:property name="base_lat_offset" value="-0.315" />
+     <xacro:property name="base_ver_offset" value="-0.178" />
+    <!-- Ground Clearance -->
+    <xacro:property name="ground_clearance" value="0.1525" />
     <!-- LiDAR Dimensions -->
      <xacro:property name="lidar_depth" value="0.098" />
+     <xacro:property name="lidar_long_offset" value="0.467" />
+     <xacro:property name="lidar_lat_offset" value="0.051" />
     <!-- Wheel Mounting Positions -->
     <xacro:property name="wheelbase" value="0.5120" />
     <xacro:property name="track" value="0.645" />
-    <xacro:property name="wheel_vertical_offset" value="0.03282" />
+    <xacro:property name="wheel_vertical_offset" value="0.204" />
+    <xacro:property name="wheel_long_offset" value="0.34"/>
     <!-- Wheel Properties for Collision -->
     <xacro:property name="wheel_length" value="0.1143" />
     <xacro:property name="wheel_radius" value="0.1651" />
+    <!-- Castor Mounting Positions -->
+    <xacro:property name="castor_vertical_offset" value="0.246" />
+    <xacro:property name="castor_long_offset" value="0.451"/>
+    <!-- Castor Visual Offsets -->
+    <xacro:property name="castor_vertical_offset_v" value="-0.135" />
+    <xacro:property name="castor_lat_offset_v" value="-0.055"/>
+    <xacro:property name="castor_long_offset_v" value="-0.044"/>
     <!-- Map -->
     <link name="map">
     </link>
-    <!-- Base link / Middle Compartment -->
+    <!-- Base link -->
     <link name="base_link">
         <visual>
+	    <origin xyz = "${base_long_offset} ${base_lat_offset} ${base_ver_offset}" rpy="0 0 0" />
             <geometry>
-                <box size="${middle_comp_length} ${middle_comp_width} ${middle_comp_height}"/>
+                <!--box size="${middle_comp_length} ${middle_comp_width} ${middle_comp_height}"/-->
+                <mesh filename="package://duda_description/meshes/base_link.stl" scale="0.001 0.001 0.001"/>
             </geometry>
             <material name="Black" />
@@ -58,42 +64,10 @@
         <parent link="map"/>
         <child link="base_link"/>
-        <origin xyz="0 0 ${middle_comp_height/2}"/>
-    </joint>
-    <!-- Front link / Front Compartment -->
-    <link name="front_link">
-        <visual>
-            <origin xyz="${front_comp_length/2} 0.0 0.0" rpy="0.0 0.0 0.0"/>
-            <geometry>
-                <box size="${front_comp_length} ${front_comp_width} ${front_comp_height}"/>
-            </geometry>
-            <material name="Blue" />
-        </visual>
-    </link>
-    <!-- Base-Front Join -->
-    <joint name="base_to_front" type="fixed">
-        <parent link="base_link"/>
-        <child link="front_link"/>
-        <origin xyz="${middle_comp_length/2} 0.0 0.0"/>
-    </joint>
-    <!-- Rear link / Rear Compartment -->
-    <link name="rear_link">
-        <visual>
-            <origin xyz="${-(rear_comp_length/2)} 0.0 0.0" rpy="0.0 0.0 0.0"/>
-            <geometry>
-                <box size="${rear_comp_length} ${rear_comp_width} ${rear_comp_height}"/>
-            </geometry>
-            <material name="Yellow" />
-        </visual>
-    </link>
-    <!-- Base-Rear Join -->
-    <joint name="base_to_rear" type="fixed">
-        <parent link="base_link"/>
-        <child link="rear_link"/>
-        <origin xyz="${-(middle_comp_length/2)} 0.0 0.0"/>
+        <origin xyz="0 0 ${(-base_ver_offset+ground_clearance)}"/>
     </joint>
     <!-- LiDAR Link -->
     <link name="lidar_link">
         <visual>
-            <origin xyz="${lidar_depth/2} 0.0 0.0" rpy="0.0 0.0 ${-radians(90)}"/>
+            <origin xyz="${lidar_depth/2} ${lidar_lat_offset} 0.0" rpy="0.0 0.0 ${-radians(90)}"/>
             <geometry>
                 <mesh filename="package://duda_description/meshes/lidar.stl" scale="0.001 0.001 0.001"/>
@@ -102,16 +76,33 @@
         </visual>
     </link>
-    <!-- front-lidar Joint -->
-    <joint name="front_to_lidar" type="fixed">
-        <parent link="front_link"/>
+    <!-- base-lidar Joint -->
+    <joint name="base_to_lidar" type="fixed">
+        <parent link="base_link"/>
         <child link="lidar_link"/>
-        <origin xyz="${front_comp_length} 0.0 0.0"/>
+        <origin xyz="${lidar_long_offset} 0.0 0.0"/>
+    </joint>
+    <!-- Castor Mount Link -->
+    <link name="castor_mount_link">
+        <visual>
+            <origin xyz="${castor_long_offset_v} ${castor_lat_offset_v} ${castor_vertical_offset_v}" rpy="0.0 0.0 0.0"/>
+            <geometry>
+                <mesh filename="package://duda_description/meshes/castor_mount.stl" scale="0.001 0.001 0.001"/>
+            </geometry>
+            <material name="Yellow" />
+        </visual>
+    </link>
+    <!-- base-castor_mount Joint -->
+    <joint name="base_to_castor_mount" type="continuous">
+        <parent link="base_link"/>
+        <child link="castor_mount_link"/>
+        <origin xyz="${-castor_long_offset} 0.0 ${base_ver_offset}"/>
+	<axis xyz="0 0 1" rpy="0 0 0" />
     </joint>
      <!-- Duda wheel macros -->
     <xacro:duda_wheel wheel_prefix="front_left">
-        <origin xyz="${front_comp_length/2} ${track/2} ${-(front_comp_height/2)}" rpy="0 0 0" />
+        <origin xyz="${wheel_long_offset} ${track/2} ${-wheel_vertical_offset}" rpy="0 0 0" />
     </xacro:duda_wheel>
     <xacro:duda_wheel wheel_prefix="front_right">
-        <origin xyz="${front_comp_length/2} ${-track/2} ${-(front_comp_height/2)}" rpy="0 0 0" />
+        <origin xyz="${wheel_long_offset} ${-track/2} ${-wheel_vertical_offset}" rpy="0 0 0" />
     </xacro:duda_wheel>
 </robot>

File: duda_robot/src/duda_description/urdf/wheel.urdf.xacro (robot description, xacro)
@@ -11,5 +11,5 @@
 				<origin xyz="0 0 0" rpy="0 0 0" />
 				<geometry>
-					<mesh filename="package://duda_description/meshes/wheel.dae" scale="0.75 0.75 0.75"/>
+					<mesh filename="package://duda_description/meshes/wheel.dae" scale="0.73 0.73 0.73"/>
 				</geometry>
 			</visual>
@@ -29,5 +29,5 @@
 		</gazebo>
 		<joint name="${wheel_prefix}_wheel" type="continuous">
-			<parent link="front_link"/>
+			<parent link="base_link"/>
 			<child link="${wheel_prefix}_wheel_link"/>
 			<xacro:insert_block name="joint_pose"/>
