Commit message: added gazebo components

File: duda_robot/src/duda_description/urdf/duda.urdf.xacro (robot description, xacro)
@@ -3,14 +3,14 @@
      <!-- Include Materials -->
      <material name="Black">
-         <color rgba="0.0 0.0 0.0 0.6"/>
+         <color rgba="0.0 0.0 0.0 0.9"/>
      </material>
      <material name="Red">
-         <color rgba="0.8 0.0 0.0 0.6"/>
+         <color rgba="0.8 0.0 0.0 0.9"/>
      </material>
     <material name="Yellow">
-         <color rgba="0.8 0.8 0.0 0.6"/>
+         <color rgba="0.8 0.8 0.0 0.9"/>
      </material>
      <material name="Blue">
-         <color rgba="0.0 0.0 0.4 0.6"/>
+         <color rgba="0.0 0.0 0.4 0.9"/>
      </material>
      <material name="White">
@@ -25,4 +25,6 @@
      <xacro:property name="base_lat_offset" value="-0.315" />
      <xacro:property name="base_ver_offset" value="-0.178" />
+    <!-- Base_Link Visual Offsets -->
+    <xacro:property name="base_link_mass" value="25" />
     <!-- Ground Clearance -->
     <xacro:property name="ground_clearance" value="0.1525" />
@@ -31,4 +33,6 @@
      <xacro:property name="lidar_long_offset" value="0.467" />
      <xacro:property name="lidar_lat_offset" value="0.051" />
+    <!-- LiDAR Mass -->
+    <xacro:property name="lidar_mass" value="" />
     <!-- Wheel Mounting Positions -->
     <xacro:property name="wheelbase" value="0.5120" />
@@ -42,15 +46,47 @@
     <xacro:property name="castor_vertical_offset" value="0.246" />
     <xacro:property name="castor_long_offset" value="0.451"/>
+    <!-- Castor Mount Mass -->
+    <xacro:property name="castor_mount_mass" value="" />
     <!-- Castor Visual Offsets -->
     <xacro:property name="castor_vertical_offset_v" value="-0.135" />
     <xacro:property name="castor_lat_offset_v" value="-0.055"/>
     <xacro:property name="castor_long_offset_v" value="-0.044"/>
+    <!-- Macro for calculating inertia of cylinder -->
+    <xacro:macro name="cylinder_inertia" params="m r h">
+        <inertia  ixx="${m*(3*r*r+h*h)/12}" ixy = "0" ixz = "0"
+                  iyy="${m*(3*r*r+h*h)/12}" iyz = "0"
+                  izz="${m*r*r/2}" />
+    </xacro:macro>
+    <!-- Macro for calculating inertia of box -->
+    <xacro:macro name="box_inertia" params="m x y z">
+        <inertia  ixx="${m*(y*y+z*z)/12}" ixy = "0" ixz = "0"
+                  iyy="${m*(x*x+z*z)/12}" iyz = "0"
+                  izz="${m*(x*x+z*z)/12}" />
+    </xacro:macro>
     <!-- Map -->
     <link name="map">
+        <inertial>
+            <mass value="0.0001" />
+            <origin xyz="0 0 0" />
+            <inertia ixx="0.0001" ixy="0.0" ixz="0.0"
+                iyy="0.0001" iyz="0.0"
+                izz="0.0001" />
+        </inertial>
+        <visual>
+            <origin xyz="0 0 0" rpy="0 0 0" />
+            <geometry>
+                <box size="0.001 0.001 0.001" />
+            </geometry>
+        </visual>
     </link>
     <!-- Base link -->
     <link name="base_link">
-        <visual>
-	    <origin xyz = "${base_long_offset} ${base_lat_offset} ${base_ver_offset}" rpy="0 0 0" />
+        <inertial>
+            <origin xyz="0.0 0.0 0.0" rpy="0.0 0.0 0.0"/>
+            <mass value="${base_link_mass}"/>
+            <box_inertia m="${base_link_mass}" x="" y="" z=""/>
+        </inertial>
+        <visual>
+	        <origin xyz = "${base_long_offset} ${base_lat_offset} ${base_ver_offset}" rpy="0 0 0" />
             <geometry>
                 <!--box size="${middle_comp_length} ${middle_comp_width} ${middle_comp_height}"/-->
@@ -59,5 +95,15 @@
             <material name="Black" />
         </visual>
-    </link>
+        <collision>
+            <origin xyz="0 0 0" rpy="0 0 0 " />
+            <geometry>
+                <mesh filename="package://duda_description/meshes/base_link.stl" scale="0.001 0.001 0.001"/>
+            </geometry>
+        </collision>
+    </link>
+    <gazebo reference="base_link">
+        <material>Gazebo/White</material>
+        <turnGravityOff>false</turnGravityOff>
+    </gazebo>
     <!-- Map to base joint -->
     <joint name="map_to_base" type="fixed">
@@ -68,4 +114,9 @@
     <!-- LiDAR Link -->
     <link name="lidar_link">
+        <inertial>
+            <mass value="${lidar_mass}" />
+            <origin xyz="0 0 0" />
+            <cylinder_inertia m="${lidar_mass}" r="${}" h="${}" />
+        </inertial>
         <visual>
             <origin xyz="${lidar_depth/2} ${lidar_lat_offset} 0.0" rpy="0.0 0.0 ${-radians(90)}"/>
@@ -75,4 +126,10 @@
             <material name="Red" />
         </visual>
+        <collision>
+            <origin xyz="0 0 0" rpy="0 0 0" />
+            <geometry>
+	            <mesh filename="package://duda_description/meshes/lidar.stl" scale="0.001 0.001 0.001"/>
+            </geometry>
+        </collision>
     </link>
     <!-- base-lidar Joint -->
@@ -82,6 +139,14 @@
         <origin xyz="${lidar_long_offset} 0.0 0.0"/>
     </joint>
+    <gazebo reference="lidar_link">
+        <turnGravityOff>false</turnGravityOff>
+    </gazebo>
     <!-- Castor Mount Link -->
     <link name="castor_mount_link">
+        <inertial>
+            <mass value="${castor_mount_mass}" />
+            <origin xyz="0 0 0" />
+            <cylinder_inertia m="${}" r="${}" h="${}" />
+        </inertial>
         <visual>
             <origin xyz="${castor_long_offset_v} ${castor_lat_offset_v} ${castor_vertical_offset_v}" rpy="0.0 0.0 0.0"/>
@@ -91,5 +156,14 @@
             <material name="Yellow" />
         </visual>
-    </link>
+        <collision>
+            <origin xyz="0 0 0" rpy="0 0 0" />
+            <geometry>
+	            <mesh filename="package://duda_description/meshes/castor_mount.stl" scale="0.001 0.001 0.001"/>
+            </geometry>
+        </collision>
+    </link>
+    <gazebo reference="caster_mount_link">
+        <turnGravityOff>false</turnGravityOff>
+    </gazebo>
     <!-- base-castor_mount Joint -->
     <joint name="base_to_castor_mount" type="continuous">
@@ -106,3 +180,27 @@
         <origin xyz="${wheel_long_offset} ${-track/2} ${-wheel_vertical_offset}" rpy="0 0 0" />
     </xacro:duda_wheel>
+    <!-- Differential drive controller  -->
+    <gazebo>
+        <plugin name="differential_drive_controller" filename="libgazebo_ros_diff_drive.so">
+            <legacyMode>true</legacyMode>
+            <rosDebugLevel>Debug</rosDebugLevel>
+            <publishWheelTF>false</publishWheelTF>
+            <robotNamespace>/</robotNamespace>
+            <publishTf>1</publishTf>
+            <publishWheelJointState>false</publishWheelJointState>
+            <alwaysOn>true</alwaysOn>
+            <updateRate>100.0</updateRate>
+            <leftJoint>front_left_wheel_joint</leftJoint>
+            <rightJoint>front_right_wheel_joint</rightJoint>
+            <wheelSeparation>${2*base_radius}</wheelSeparation>
+            <wheelDiameter>${2*wheel_radius}</wheelDiameter>
+            <broadcastTF>1</broadcastTF>
+            <wheelTorque>30</wheelTorque>
+            <wheelAcceleration>1.8</wheelAcceleration>
+            <commandTopic>cmd_vel</commandTopic>
+            <odometryFrame>odom</odometryFrame>
+            <odometryTopic>odom</odometryTopic>
+            <robotBaseFrame>base_footprint</robotBaseFrame>
+        </plugin>
+    </gazebo>
 </robot>

Commit message: deleting useless files

File: duda_robot/src/duda_description/urdf/duda.urdf.xacro (robot description, xacro)
@@ -25,6 +25,9 @@
      <xacro:property name="base_lat_offset" value="-0.315" />
      <xacro:property name="base_ver_offset" value="-0.178" />
-    <!-- Base_Link Visual Offsets -->
+    <!-- Base_Link Properties -->
     <xacro:property name="base_link_mass" value="25" />
+    <xacro:property name="base_link_x" value="1.22" />
+    <xacro:property name="base_link_y" value="0.633" />
+    <xacro:property name="base_link_x" value="0.356" />
     <!-- Ground Clearance -->
     <xacro:property name="ground_clearance" value="0.1525" />
@@ -33,6 +36,19 @@
      <xacro:property name="lidar_long_offset" value="0.467" />
      <xacro:property name="lidar_lat_offset" value="0.051" />
-    <!-- LiDAR Mass -->
-    <xacro:property name="lidar_mass" value="" />
+    <!-- LiDAR properties -->
+    <xacro:property name="lidar_mass" value="1.5" />
+    <xacro:property name="lidar_x" value="0.106" />
+    <xacro:property name="lidar_y" value="0.102" />
+    <xacro:property name="lidar_z" value="0.162" />
+    <!-- GPS Properties -->
+    <xacro:property name="gps_mass" value="1.2" />
+    <xacro:property name="gps_x" value="0.16" />
+    <xacro:property name="gps_y" value="0.16" />
+    <xacro:property name="gps_z" value="0.10" />
+    <!-- IMU Properties -->
+    <xacro:property name="imu_mass" value="0.3" />
+    <xacro:property name="imu_x" value="0.077" />
+    <xacro:property name="imu_y" value="0.276" />
+    <xacro:property name="imu_z" value="0.037" />
     <!-- Wheel Mounting Positions -->
     <xacro:property name="wheelbase" value="0.5120" />
@@ -40,12 +56,19 @@
     <xacro:property name="wheel_vertical_offset" value="0.204" />
     <xacro:property name="wheel_long_offset" value="0.34"/>
-    <!-- Wheel Properties for Collision -->
-    <xacro:property name="wheel_length" value="0.1143" />
-    <xacro:property name="wheel_radius" value="0.1651" />
+    <!-- Wheel Properties -->
+    <xacro:property name="wheel_length" value="0.065" />
+    <xacro:property name="wheel_radius" value="0.254" />
     <!-- Castor Mounting Positions -->
     <xacro:property name="castor_vertical_offset" value="0.246" />
     <xacro:property name="castor_long_offset" value="0.451"/>
-    <!-- Castor Mount Mass -->
-    <xacro:property name="castor_mount_mass" value="" />
+    <!-- Castor Mount Properties -->
+    <xacro:property name="castor_mount_mass" value="7" />
+    <xacro:property name="castor_mount_x" value="0.944" />
+    <xacro:property name="castor_mount_y" value="0.111" />
+    <xacro:property name="castor_mount_z" value="0.135" />
+    <!-- Caster Wheel Properties -->
+    <xacro:property name="castor_wheel_mass" value="1">
+    <xacro:property name="castor_wheel_radius" value="0.050">
+    <xacro:property name="castor_wheel_length" value="0.030">
     <!-- Castor Visual Offsets -->
     <xacro:property name="castor_vertical_offset_v" value="-0.135" />
