Commit message: added camera mast

File: duda_robot/src/duda_description/urdf/duda.urdf.xacro (robot description, xacro)
@@ -21,4 +21,5 @@
     <!--Include URDF/XACRO files -->
     <xacro:include filename="$(find duda_description)/urdf/wheel.urdf.xacro" />
+    <xacro:include filename="$(find duda_description)/urdf/camera_mast.urdf.xacro" />
     <!-- Constants -->
     <xacro:property name="M_PI" value="3.14159" />
@@ -78,4 +79,11 @@
     <xacro:property name="castor_lat_offset_v" value="-0.055" />
     <xacro:property name="castor_long_offset_v" value="-0.044" />
+    <!-- Camera Mast Properties -->
+	<xacro:property name="camera_mast_vertical_mass" value="0.8" />
+	<xacro:property name="camera_mast_horizontal_mass" value="0.4" />
+	<xacro:property name="camera_mast_cross_section_size" value="0.02" />
+	<xacro:property name="camera_mast_long_offset" value="0.24" />
+    <xacro:property name="camera_mast_height" value="0.100" />
+    <xacro:property name="camera_mast_separation" value="0.04" />
     <!-- Macro for calculating inertia of cylinder -->
     <xacro:macro name="cylinder_inertia" params="m r h">
@@ -243,4 +251,6 @@
         <turnGravityOff>false</turnGravityOff>
     </gazebo>
+    <!-- Camera mast macros -->
+    <xacro:camera_mast height="${camera_mast_height}" separation="${camera_mast_separation}" />
     <!-- Duda wheel macros -->
     <xacro:duda_wheel wheel_prefix="front_left">

Commit message: added camera link

File: duda_robot/src/duda_description/urdf/duda.urdf.xacro (robot description, xacro)
@@ -80,10 +80,12 @@
     <xacro:property name="castor_long_offset_v" value="-0.044" />
     <!-- Camera Mast Properties -->
-	<xacro:property name="camera_mast_vertical_mass" value="0.8" />
-	<xacro:property name="camera_mast_horizontal_mass" value="0.4" />
-	<xacro:property name="camera_mast_cross_section_size" value="0.02" />
-	<xacro:property name="camera_mast_long_offset" value="0.24" />
+    <xacro:property name="camera_mast_vertical_mass" value="0.8" />
+    <xacro:property name="camera_mast_horizontal_mass" value="0.4" />
+    <xacro:property name="camera_mast_cross_section_size" value="0.02" />
+    <xacro:property name="camera_mast_long_offset" value="0.24" />
     <xacro:property name="camera_mast_height" value="0.6" />
     <xacro:property name="camera_mast_separation" value="0.6" />
+    <!-- Camera Properties -->
+    <xacro:property name="camera_size" value="0.05" />
     <!-- Macro for calculating inertia of cylinder -->
     <xacro:macro name="cylinder_inertia" params="m r h">
@@ -220,5 +222,5 @@
         <axis xyz="0 0 1" rpy="0 0 0" />
     </joint>
-	<!-- Castor Wheel Link -->
+    <!-- Castor Wheel Link -->
     <link name="castor_wheel_link">
     <inertial>
@@ -253,4 +255,31 @@
     <!-- Camera mast macros -->
     <xacro:camera_mast height="${camera_mast_height}" separation="${camera_mast_separation}" />
+    <!-- Camera Link -->
+    <link name="camera_link">
+    <collision>
+        <origin xyz="0 0 0" rpy="0 0 0" />
+        <geometry>
+            <box size="${camera_size} ${camera_size} ${camera_size}" />
+        </geometry>
+    </collision>
+    <visual>
+        <origin xyz="0 0 0" rpy="0 0 0" />
+        <geometry>
+            <box size="${camera_size} ${camera_size} ${camera_size}" />
+        </geometry>
+        <material name="Black" />
+    </visual>
+    <joint name="camera_mast_to_camera" type="fixed">
+        <axis xyz="0 1 0" />
+        <origin xyz="${camera_mast_cross_section_size/2} 0 0" rpy="0 0 0"/>
+        <parent link="camera_mast_horizontal_link"/>
+        <child link="camera_link"/>
+    </joint>
+    <inertial>
+        <mass value="1e-5" />
+        <origin xyz="0 0 0" rpy="0 0 0" />
+        <inertia ixx="1e-6" ixy="0" ixz="0" iyy="1e-6" iyz="0" izz="1e-6" />
+    </inertial>
+    </link>
     <!-- Duda wheel macros -->
     <xacro:duda_wheel wheel_prefix="front_left">

Commit message: added camera link and its joint

File: duda_robot/src/duda_description/urdf/duda.urdf.xacro (robot description, xacro)
@@ -270,10 +270,4 @@
         <material name="Black" />
     </visual>
-    <joint name="camera_mast_to_camera" type="fixed">
-        <axis xyz="0 1 0" />
-        <origin xyz="${camera_mast_cross_section_size/2} 0 0" rpy="0 0 0"/>
-        <parent link="camera_mast_horizontal_link"/>
-        <child link="camera_link"/>
-    </joint>
     <inertial>
         <mass value="1e-5" />
@@ -282,4 +276,11 @@
     </inertial>
     </link>
+    <!-- Camera mast to Camera Joint -->
+    <joint name="camera_mast_to_camera" type="fixed">
+        <axis xyz="0 1 0" />
+        <origin xyz="${camera_mast_cross_section_size/2} 0 0" rpy="0 0 0" />
+        <parent link="camera_mast_horizontal_link" />
+        <child link="camera_link" />
+    </joint>
     <!-- Duda wheel macros -->
     <xacro:duda_wheel wheel_prefix="front_left">

Commit message: added camera link and joint

File: duda_robot/src/duda_description/urdf/duda.urdf.xacro (robot description, xacro)
@@ -278,5 +278,4 @@
     <!-- Camera mast to Camera Joint -->
     <joint name="camera_mast_to_camera" type="fixed">
-        <axis xyz="0 1 0" />
         <origin xyz="${camera_mast_cross_section_size/2} 0 0" rpy="0 0 0" />
         <parent link="camera_mast_horizontal_link" />

Commit message: added teleop

File: duda_robot/src/duda_description/urdf/duda.urdf.xacro (robot description, xacro)
@@ -58,5 +58,5 @@
     <xacro:property name="track" value="0.645" />
     <xacro:property name="wheel_vertical_offset" value="0.204" />
-    <xacro:property name="wheel_long_offset" value="0.34" />
+    <xacro:property name="wheel_long_offset" value="0.37" />
     <!-- Wheel Properties -->
     <xacro:property name="wheel_length" value="0.065" />
@@ -347,9 +347,8 @@
             <broadcastTF>1</broadcastTF>
             <wheelTorque>30</wheelTorque>
-            <wheelAcceleration>1.8</wheelAcceleration>
             <commandTopic>cmd_vel</commandTopic>
             <odometryFrame>odom</odometryFrame>
             <odometryTopic>odom</odometryTopic>
-            <robotBaseFrame>base_footprint</robotBaseFrame>
+            <robotBaseFrame>map</robotBaseFrame>
         </plugin>
     </gazebo>

Commit message: added imu and gps with gazebo plugins

File: duda_robot/src/duda_description/urdf/duda.urdf.xacro (robot description, xacro)
@@ -9,4 +9,7 @@
     <material name="Red">
         <color rgba="0.8 0.0 0.0 0.9" />
+    </material>
+    <material name="Orange">
+        <color rgba="1 0.64 0.0 0.9" />
     </material>
     <material name="Yellow">
@@ -49,9 +52,15 @@
     <xacro:property name="gps_y" value="0.16" />
     <xacro:property name="gps_z" value="0.10" />
+    <xacro:property name="gps_long_offset" value="0.36" />
+    <xacro:property name="gps_lat_offset" value="0" />
+    <xacro:property name="gps_vertical_offset" value="0.2" />
     <!-- IMU Properties -->
     <xacro:property name="imu_mass" value="0.3" />
-    <xacro:property name="imu_x" value="0.077" />
-    <xacro:property name="imu_y" value="0.276" />
-    <xacro:property name="imu_z" value="0.037" />
+    <xacro:property name="imu_x" value="0.03" />
+    <xacro:property name="imu_y" value="0.04" />
+    <xacro:property name="imu_z" value="0.015" />
+    <xacro:property name="imu_long_offset" value="0.2" />
+    <xacro:property name="imu_lat_offset" value="0.15" />
+    <xacro:property name="imu_vertical_offset" value="0.15" />
     <!-- Wheel Mounting Positions -->
     <xacro:property name="wheelbase" value="0.5120" />
@@ -191,4 +200,76 @@
         </sensor>
     </gazebo>
+    <!-- IMU Link -->
+    <link name="imu_link">
+    <inertial>
+        <mass value="${imu_mass}" />
+        <box_inertia m="${imu_mass}" x="${imu_x}" y="${imu_y}" z="${imu_z}">
+    </inertial>
+    <visual>
+        <origin xyz="0 0 ${imu_z/2}" rpy="0 0 0" />
+        <box size="${imu_x} ${imu_y} ${imu_z}" />
+        <material name="White">
+    </visual>
+    </link>
+    <!-- Base to IMU Joint -->
+    <joint name="base_to_imu" type="fixed">
+        <origin xyz="${imu_long_offset} ${imu_lat_offset} ${imu_vertical_offset}" rpy="0.0 0.0 0.0" />
+        <parent link="base_link" />
+        <child link="imu_link" />
+    </joint>
+    <!-- IMU Gazebo Plugin -->
+    <gazebo reference="imu_link">
+        <gravity>true</gravity>
+        <sensor name="imu_sensor" type="imu">
+            <always_on>true</always_on>
+            <update_rate>100</update_rate>
+            <visualize>true</visualize>
+            <topic>__default_topic__</topic>
+            <plugin filename="libgazebo_ros_imu_sensor.so" name="imu_plugin">
+                <topicName>imu</topicName>
+                <bodyName>imu_link</bodyName>
+                <updateRateHZ>50.0</updateRateHZ>
+                <gaussianNoise>0.0</gaussianNoise>
+                <xyzOffset>0 0 0</xyzOffset>
+                <rpyOffset>0 0 0</rpyOffset>
+                <frameName>imu_link</frameName>
+            </plugin>
+            <pose>0 0 0 0 0 0</pose>
+        </sensor>
+    </gazebo>
+    <!-- GPS Link -->
+    <link name="gps_link">
+    <inertial>
+        <mass value="${gps_mass}" />
+        <box_inertia m="${gps_mass}" x="${gps_x}" y="${gps_y}" z="${gps_z}">
+    </inertial>
+    <visual>
+        <origin xyz="0 0 0" rpy="0 0 0" />
+        <box size="${gps_x} ${gps_y} ${gps_z}" />
+        <material name="Orange">
+    </visual>
+    </link>
+    <!-- Base to GPS Joint -->
+    <joint name="base_to_gps" type="fixed">
+        <origin xyz="${gps_long_offset} ${gps_lat_offset} ${gps_vertical_offset}" rpy="0.0 0.0 0.0" />
+        <parent link="base_link" />
+        <child link="imu_link" />
+    </joint>
+    <!-- GPS Gazebo Plugin -->
+    <gazebo>
+        <plugin name="gps_controller" filename="libhector_gazebo_ros_gps.so">
+            <robotNamespace>/</robotNamespace>
+            <updateRate>40</updateRate>
+            <bodyName>base_link</bodyName>
+            <frameId>base_link</frameId>
+            <topicName>navsat/fix</topicName>
+            <velocityTopicName>navsat/vel</velocityTopicName>
+            <referenceLatitude>49.9</referenceLatitude>
+            <referenceLongitude>8.9</referenceLongitude>
+            <referenceHeading>0</referenceHeading>
+            <referenceAltitude>0</referenceAltitude>
+            <drift>0.0001 0.0001 0.0001</drift>
+        </plugin>
+    </gazebo>
     <!-- Castor Mount Link -->
     <link name="castor_mount_link">
@@ -244,4 +325,5 @@
     </collision>
     </link>
+    <!-- Castor mount to castor wheel Joint -->
     <joint name="castor_mount_to_castor_wheel" type="continuous">
         <parent link="castor_mount_link" />
@@ -345,4 +427,5 @@
             <wheelSeparation>${track}</wheelSeparation>
             <wheelDiameter>${2*wheel_radius}</wheelDiameter>
+            <wheelAcceleration>1.8</wheelAcceleration>
             <broadcastTF>1</broadcastTF>
             <wheelTorque>30</wheelTorque>

Commit message: resolved constant motion problem and fixed imu and gps

File: duda_robot/src/duda_description/urdf/duda.urdf.xacro (robot description, xacro)
@@ -51,8 +51,8 @@
     <xacro:property name="gps_x" value="0.16" />
     <xacro:property name="gps_y" value="0.16" />
-    <xacro:property name="gps_z" value="0.10" />
-    <xacro:property name="gps_long_offset" value="0.36" />
+    <xacro:property name="gps_z" value="0.08" />
+    <xacro:property name="gps_long_offset" value="0.41" />
     <xacro:property name="gps_lat_offset" value="0" />
-    <xacro:property name="gps_vertical_offset" value="0.2" />
+    <xacro:property name="gps_vertical_offset" value="0.19" />
     <!-- IMU Properties -->
     <xacro:property name="imu_mass" value="0.3" />
@@ -60,7 +60,7 @@
     <xacro:property name="imu_y" value="0.04" />
     <xacro:property name="imu_z" value="0.015" />
-    <xacro:property name="imu_long_offset" value="0.2" />
+    <xacro:property name="imu_long_offset" value="0.3" />
     <xacro:property name="imu_lat_offset" value="0.15" />
-    <xacro:property name="imu_vertical_offset" value="0.15" />
+    <xacro:property name="imu_vertical_offset" value="0.07" />
     <!-- Wheel Mounting Positions -->
     <xacro:property name="wheelbase" value="0.5120" />
@@ -76,12 +76,12 @@
     <!-- Castor Mount Properties -->
     <xacro:property name="castor_mount_mass" value="7" />
-    <xacro:property name="castor_mount_x" value="0.944" />
+    <xacro:property name="castor_mount_x" value="0.094" />
     <xacro:property name="castor_mount_y" value="0.111" />
     <xacro:property name="castor_mount_z" value="0.135" />
-    <!-- Caster Wheel Properties -->
+    <!-- Castor Wheel Properties -->
     <xacro:property name="castor_wheel_mass" value="1" />
     <xacro:property name="castor_wheel_radius" value="0.050" />
     <xacro:property name="castor_wheel_length" value="0.030" />
-    <xacro:property name="castor_wheel_vertical_offset" value="0.1" />
+    <xacro:property name="castor_wheel_vertical_offset" value="0.12" />
     <!-- Castor Visual Offsets -->
     <xacro:property name="castor_vertical_offset_v" value="-0.135" />
@@ -177,5 +177,5 @@
         <sensor type="ray" name="head_hokuyo_sensor">
             <pose>0 0 0 0 0 0</pose>
-            <visualize>true</visualize>
+            <visualize>false</visualize>
             <update_rate>40</update_rate>
             <ray>
@@ -204,15 +204,17 @@
     <inertial>
         <mass value="${imu_mass}" />
-        <box_inertia m="${imu_mass}" x="${imu_x}" y="${imu_y}" z="${imu_z}">
-    </inertial>
-    <visual>
-        <origin xyz="0 0 ${imu_z/2}" rpy="0 0 0" />
-        <box size="${imu_x} ${imu_y} ${imu_z}" />
-        <material name="White">
+        <box_inertia m="${imu_mass}" x="${imu_x}" y="${imu_x}" z="${imu_z}" />
+    </inertial>
+    <visual>
+        <origin xyz="0 0 0" rpy="0 0 0" />
+        <geometry>
+            <box size="${imu_x} ${imu_x} ${imu_z}" />
+        </geometry>
+        <material name="White" />
     </visual>
     </link>
     <!-- Base to IMU Joint -->
     <joint name="base_to_imu" type="fixed">
-        <origin xyz="${imu_long_offset} ${imu_lat_offset} ${imu_vertical_offset}" rpy="0.0 0.0 0.0" />
+        <origin xyz="0 0 0" rpy="0.0 0.0 0.0" />
         <parent link="base_link" />
         <child link="imu_link" />
@@ -220,18 +222,20 @@
     <!-- IMU Gazebo Plugin -->
     <gazebo reference="imu_link">
+        <material>Gazebo/Black</material>
+        <turnGravityOff>false</turnGravityOff>
         <gravity>true</gravity>
         <sensor name="imu_sensor" type="imu">
             <always_on>true</always_on>
-            <update_rate>100</update_rate>
+            <update_rate>50</update_rate>
             <visualize>true</visualize>
             <topic>__default_topic__</topic>
             <plugin filename="libgazebo_ros_imu_sensor.so" name="imu_plugin">
                 <topicName>imu</topicName>
-                <bodyName>imu_link</bodyName>
+                <bodyName>map</bodyName>
                 <updateRateHZ>50.0</updateRateHZ>
                 <gaussianNoise>0.0</gaussianNoise>
                 <xyzOffset>0 0 0</xyzOffset>
                 <rpyOffset>0 0 0</rpyOffset>
-                <frameName>imu_link</frameName>
+                <frameName>map</frameName>
             </plugin>
             <pose>0 0 0 0 0 0</pose>
@@ -242,10 +246,12 @@
     <inertial>
         <mass value="${gps_mass}" />
-        <box_inertia m="${gps_mass}" x="${gps_x}" y="${gps_y}" z="${gps_z}">
-    </inertial>
-    <visual>
-        <origin xyz="0 0 0" rpy="0 0 0" />
-        <box size="${gps_x} ${gps_y} ${gps_z}" />
-        <material name="Orange">
+        <box_inertia m="${gps_mass}" x="${gps_x}" y="${gps_y}" z="${gps_z}" />
+    </inertial>
+    <visual>
+        <origin xyz="0 0 0" rpy="0 0 0" />
+        <geometry>
+            <box size="${gps_x} ${gps_y} ${gps_z}" />
+        </geometry>
+        <material name="Orange" />
     </visual>
     </link>
@@ -254,8 +260,10 @@
         <origin xyz="${gps_long_offset} ${gps_lat_offset} ${gps_vertical_offset}" rpy="0.0 0.0 0.0" />
         <parent link="base_link" />
-        <child link="imu_link" />
+        <child link="gps_link" />
     </joint>
     <!-- GPS Gazebo Plugin -->
-    <gazebo>
+    <gazebo reference="gps_link">
+        <material>Gazebo/Orange</material>
+        <turnGravityOff>false</turnGravityOff>
         <plugin name="gps_controller" filename="libhector_gazebo_ros_gps.so">
             <robotNamespace>/</robotNamespace>
@@ -307,5 +315,5 @@
     <link name="castor_wheel_link">
     <inertial>
-        <origin xyz="0.0 0.0 0.0" rpy="0.0 0.0 0.0" />
+        <origin xyz="0.0 0.0 0.0" rpy="${radians(90)} 0.0 0.0" />
         <mass value="${castor_wheel_mass}" />
         <cylinder_inertia m="${castor_wheel_mass}" r="${castor_wheel_radius}" h="${castor_wheel_length}" />
@@ -412,5 +420,5 @@
         <origin xyz="${wheel_long_offset} ${-track/2} ${-wheel_vertical_offset}" rpy="0 0 0" />
     </xacro:duda_wheel>
-    <!-- Differential drive controller Gazebo Plugin -->
+    <!-- Differential drive controller Gazebo Plugin >
     <gazebo>
         <plugin name="differential_drive_controller" filename="libgazebo_ros_diff_drive.so">
@@ -435,4 +443,4 @@
             <robotBaseFrame>map</robotBaseFrame>
         </plugin>
-    </gazebo>
+    </gazebo -->
 </robot>

File: duda_robot/src/duda_description/urdf/wheel.urdf.xacro (robot description, xacro)
@@ -22,6 +22,6 @@
 		</link>
 		<gazebo reference="${wheel_prefix}_wheel_link">
-			<mu1 value="1.0"/>
-			<mu2 value="1.0"/>
+			<mu1 value="3.0"/>
+			<mu2 value="3.0"/>
 			<kp value="10000000.0" />
 			<kd value="1.0" />

Commit message: trying alternative imu

File: duda_robot/src/duda_description/urdf/duda.urdf.xacro (robot description, xacro)
@@ -221,24 +221,13 @@
     </joint>
     <!-- IMU Gazebo Plugin -->
-    <gazebo reference="imu_link">
-        <material>Gazebo/Black</material>
-        <turnGravityOff>false</turnGravityOff>
-        <gravity>true</gravity>
-        <sensor name="imu_sensor" type="imu">
-            <always_on>true</always_on>
-            <update_rate>50</update_rate>
-            <visualize>true</visualize>
-            <topic>__default_topic__</topic>
-            <plugin filename="libgazebo_ros_imu_sensor.so" name="imu_plugin">
-                <topicName>imu</topicName>
-                <bodyName>map</bodyName>
-                <updateRateHZ>50.0</updateRateHZ>
-                <gaussianNoise>0.0</gaussianNoise>
-                <xyzOffset>0 0 0</xyzOffset>
-                <rpyOffset>0 0 0</rpyOffset>
-                <frameName>map</frameName>
-            </plugin>
-            <pose>0 0 0 0 0 0</pose>
-        </sensor>
+    <gazebo>
+        <plugin name="imu_plugin" filename="libgazebo_ros_imu.so">
+            <alwaysOn>true</alwaysOn>
+            <bodyName>map</bodyName>
+            <topicName>imu</topicName>
+            <serviceName>imu_service</serviceName>
+            <gaussianNoise>0.0</gaussianNoise>
+            <updateRate>20.0</updateRate>
+        </plugin>
     </gazebo>
     <!-- GPS Link -->

Commit message: added robot pose publisher package

File: duda_robot/src/duda_description/urdf/duda.urdf.xacro (robot description, xacro)
@@ -83,5 +83,5 @@
     <xacro:property name="castor_wheel_radius" value="0.050" />
     <xacro:property name="castor_wheel_length" value="0.030" />
-    <xacro:property name="castor_wheel_vertical_offset" value="0.12" />
+    <xacro:property name="castor_wheel_vertical_offset" value="0.11" />
     <!-- Castor Visual Offsets -->
     <xacro:property name="castor_vertical_offset_v" value="-0.135" />
@@ -144,10 +144,10 @@
         <turnGravityOff>false</turnGravityOff>
     </gazebo>
-    <!-- Map to base joint -->
+    <!-- Map to base joint >
     <joint name="map_to_base" type="fixed">
         <parent link="map" />
         <child link="base_link" />
         <origin xyz="0 0 ${(-base_ver_offset+ground_clearance)}" />
-    </joint>
+    </joint-->
     <!-- LiDAR Link -->
     <link name="lidar_link">

Commit message: diff_drive_control working , changed mu $ wTorque

File: duda_robot/src/duda_description/urdf/duda.urdf.xacro (robot description, xacro)
@@ -144,10 +144,10 @@
         <turnGravityOff>false</turnGravityOff>
     </gazebo>
-    <!-- Map to base joint >
+    <!-- Map to base joint -->
     <joint name="map_to_base" type="fixed">
         <parent link="map" />
         <child link="base_link" />
         <origin xyz="0 0 ${(-base_ver_offset+ground_clearance)}" />
-    </joint-->
+    </joint>
     <!-- LiDAR Link -->
     <link name="lidar_link">
@@ -295,5 +295,5 @@
     </gazebo>
     <!-- base-castor_mount Joint -->
-    <joint name="base_to_castor_mount" type="continuous">
+    <joint name="base_to_castor_mount" type="fixed">
         <parent link="base_link" />
         <child link="castor_mount_link" />
@@ -409,5 +409,5 @@
         <origin xyz="${wheel_long_offset} ${-track/2} ${-wheel_vertical_offset}" rpy="0 0 0" />
     </xacro:duda_wheel>
-    <!-- Differential drive controller Gazebo Plugin >
+    <!-- Differential drive controller Gazebo Plugin -->
     <gazebo>
         <plugin name="differential_drive_controller" filename="libgazebo_ros_diff_drive.so">
@@ -420,11 +420,11 @@
             <alwaysOn>true</alwaysOn>
             <updateRate>100.0</updateRate>
-            <leftJoint>front_left_wheel_joint</leftJoint>
-            <rightJoint>front_right_wheel_joint</rightJoint>
+            <leftJoint>front_left_wheel</leftJoint>
+            <rightJoint>front_right_wheel</rightJoint>
             <wheelSeparation>${track}</wheelSeparation>
             <wheelDiameter>${2*wheel_radius}</wheelDiameter>
             <wheelAcceleration>1.8</wheelAcceleration>
             <broadcastTF>1</broadcastTF>
-            <wheelTorque>30</wheelTorque>
+            <wheelTorque>180</wheelTorque>
             <commandTopic>cmd_vel</commandTopic>
             <odometryFrame>odom</odometryFrame>
@@ -432,4 +432,4 @@
             <robotBaseFrame>map</robotBaseFrame>
         </plugin>
-    </gazebo -->
+    </gazebo>
 </robot>

File: duda_robot/src/duda_description/urdf/wheel.urdf.xacro (robot description, xacro)
@@ -22,6 +22,6 @@
 		</link>
 		<gazebo reference="${wheel_prefix}_wheel_link">
-			<mu1 value="3.0"/>
-			<mu2 value="3.0"/>
+			<mu1 value="100000.0"/>
+			<mu2 value="100000.0"/>
 			<kp value="10000000.0" />
 			<kd value="1.0" />
